File: Hardware/PCBA/-A/Occupancy_Sensor-A/Occupancy_Sensor-A.kicad_sch (KiCad schematic)
At the start: 60 parts, among them J1 USB_C_Receptacle, J2 Conn_02x05_Odd_Even, Q1 2N7002, Q2 2N7002, SW1 SW_Push, SW2 SW_SPDT, U1 TPS78318DDCR, U3 TPS562200, U4 STM32WB55CGUx, U6 ECMF02-2AMX6, Y1 Crystal_GND24_Small, Y2 Crystal_GND24_Small

Commit message: Add TOF footprint, component to schematic
Parts:
- removed C16, C17: 1u, Capacitor_SMD:C_0402_1005Metric, symbol Device:C
- removed C19, C20: 22u, Capacitor_SMD:C_0402_1005Metric, symbol Device:C
- removed C21: 10u, Capacitor_SMD:C_0402_1005Metric, symbol Device:C
- removed C22, C23, C24: 100n, Capacitor_SMD:C_0402_1005Metric, symbol Device:C_Small
- removed L2: 3.3u, Inductor_SMD:L_Sumida_CDMC6D28_7.25x6.5mm, symbol Device:L
- removed R1: 10K, Resistor_SMD:R_0402_1005Metric, symbol Device:R
- removed R5: 22R, Resistor_SMD:R_0402_1005Metric, symbol Device:R
- removed R6: 2.2K, Resistor_SMD:R_0402_1005Metric, symbol Device:R
- removed U1: TPS78318DDCR, Package_TO_SOT_SMD:SOT-23-5, symbol TPS78318DDCR:TPS78318DDCR
- removed U2: ~, Occupancy_Sensor_Custom_Footprints:TCS3430, symbol TCS3430:TCS3430
- removed U3: TPS562200, Package_TO_SOT_SMD:SOT-23-6, symbol Regulator_Switching:TPS562200
- added C16, C17: 100n, Capacitor_SMD:C_0402_1005Metric, symbol Device:C_Small
- added C27, C29, C30, C31: 1u, Capacitor_SMD:C_0402_1005Metric, symbol Device:C
- added Q3, Q4, Q5: 2N7002, Package_TO_SOT_SMD:SOT-23, symbol Transistor_FET:2N7002
- added R16, R17: 47K, Resistor_SMD:R_0402_1005Metric, symbol Device:R
- added R20, R21, R22, R23, R24, R25: 2.2K, Resistor_SMD:R_0402_1005Metric, symbol Device:R
- added U1: TCS3430, Occupancy_Sensor_Custom_Footprints:TCS3430, symbol Occupancy_Sensor_Custom_Symbols:TCS3430
- added U2: VL53L8CX, Occupancy_Sensor_Custom_Footprints:VL53L8CX, symbol Occupancy_Sensor_Custom_Symbols:VL53L8CX
- added U8: TPS7A03185PDQNR, Package_TO_SOT_SMD:SOT-23-5, symbol Occupancy_Sensor_Custom_Symbols:TPS7A03185PDBVR
- added U9: TPS7A0333PDBVR, Package_TO_SOT_SMD:SOT-23-5, symbol Occupancy_Sensor_Custom_Symbols:TPS7A0333PDBVR
- C18: value 10u -> 1u
- C5: value 2.2u -> 4.7u
- R10, R3: value 10K -> 40K
- R2, R4: value 10K -> 47K
- R7, R8: value 2.2K -> 47K
- R9: value 33.2K -> 47K
Connections:
- net +1V8: now also C18.1, C16.1, C17.1, C29.1, Q3.1 (G), Q4.1 (G), Q5.1 (G), R16.1, R20.1, R22.1, R24.1, U1.1 (VDD), U2.A3 (IOVDD), U2.B7 (CORE_1V8), U8.5 (OUT); no longer C5.1, R2.1, R8.1
- net +3.3V: now also C5.1, R8.1, C31.1, R17.1, R21.1, R23.1, R25.1, U2.C4 (AVDD), U9.5 (OUT); no longer R9.1
- net 1V8_EN: now also U8.3 (EN)
- net GND: now also R2.2, R4.2, R9.2, C16.2, C17.2, C27.2, C29.2, C30.2, C31.2, U1.7 (GND), U1.8 (GND), U2.A6 (RSVD1), U2.A7 (RSVD2), U2.B4 (PAD), U2.C3 (GND), U2.C6 (RSVD3), U2.C7 (GND), U8.2 (GND), U9.2 (GND); no longer R10.2
- net SCL_1V8: now also Q2.2 (S), R22.2, U1.3 (SCL), U2.A5 (SCL/MCLK); no longer Q1.2 (S), R7.2
- net SDA_1V8: now also Q4.2 (S), R24.2, U1.2 (SDA), U2.A4 (SDA/MOSI); no longer Q2.2 (S), R2.2
- net VBUS: now also C27.1, C30.1, U8.1 (IN), U9.1 (IN), U9.3 (EN); no longer C18.1
- net SYNC_3V3: now reaches R8.2
- net SYNC_3V3: now also Q3.3 (D)
- net I2C_RST: now reaches R10.1
- net I2C_RST: no longer R9.2
- net +3V3 renamed LPn
- net LPn: no longer R4.1
- net SCL renamed INT_CLR
- net INT_CLR: now also R21.2; no longer R3.2
- net SDA renamed SCL_3V3
- net SCL_3V3: now also R23.2; no longer R4.2
- new net: R2.1, U2.C1 (SPI_I2C_N)
- new net I2C_RST_1V8: R10.2, R9.1, U2.C2 (NCS)
- new net INT_CLR_1V8: Q1.2 (S), R20.2, U1.4 (INT)
- new net INT_TOF: Q5.3 (D), R17.2
- new net INT_TOF_1V8: Q5.2 (S), R16.2, U2.A1 (INT)
- new net LPn_1V8: R3.2, R4.1, U2.A2 (LPn)
- new net SDA_3V3: Q4.3 (D), R25.2
- new net SYNC_1V8: Q3.2 (S), R7.2, U2.B1 (SYNC)
- no-connect marks 14 -> 15
Other:
- note added: "Depop FET and 3V3-side pullup if SYNC not used"
- note added: "I2C Reset active high Voltage divider ensures 1.8V and required 47K pulldown"
- note added: "MICROCONTROLLER"
- note added: "REGULATORS"
- note added: "TCS340 COLOR SENSOR"
- note added: "USB"
- note added: "VL53L8 TOF SENSOR"

Commit message: Update antenna circuit
Parts:
- renumbered C5 to C1, C6 to C10, C7 to C11, C14 to C12, C4 to C13, C15 to C14, C8 to C15, C1 to C16, C10 to C17, C2 to C18, C9 to C19, C17 to C2, C3 to C20, C13 to C21, C11 to C22, C12 to C23, C30 to C3, C16 to C4, C31 to C5, C27 to C6, C29 to C7, C18 to C8, C25 to C9, D3 to D1, D1 to D3, L3 to L2, Q5 to Q1, Q3 to Q2, Q1 to Q3, Q2 to Q4, Q4 to Q5, R11 to R1, R8 to R10, R3 to R11, R4 to R12, R20 to R14, R22 to R16, R21 to R17, R23 to R18, R24 to R19, R12 to R2, R25 to R20, R2 to R3, R10 to R4, R9 to R5, R16 to R6, R14 to R8, R17 to R9, SW2 to SW1, SW1 to SW2, U9 to U1, U6 to U3, U8 to U4, U1 to U5, U4 to U6
